Commit message: Added a few changes that (1) Only builds modules needed for Gazebo and Rviz while ignoring ethercat-related packages, (2) Add C++11 for Gazebo plugin, (3) Add color to hand in Gazebo

File: robotiq_s_model_visualization/cfg/robotiq_hand_macro.urdf.xacro (robot description, xacro)
@@ -630,4 +630,44 @@
     <gazebo reference="${prefix}link_paraproximal_bar_paramedian_hinge_couple">
       <implicitSpringDamper>1</implicitSpringDamper>
+    </gazebo>
+    <!-- Added: Color in Gazebo visualization -->
+    <gazebo reference="${prefix}link_0">
+      <material>Gazebo/Black</material>
+    </gazebo>
+    <gazebo reference="${prefix}link_1">
+      <material>Gazebo/Black</material>
+    </gazebo>
+    <gazebo reference="${prefix}link_2">
+      <material>Gazebo/Black</material>
+    </gazebo>
+    <gazebo reference="${prefix}link_3">
+      <material>Gazebo/Black</material>
+    </gazebo>
+    <gazebo reference="${prefix}link_proximal_actuating_hinge">
+      <material>Gazebo/Black</material>
+    </gazebo>
+    <gazebo reference="${prefix}link_paraproximal_actuating_hinge">
+      <material>Gazebo/Black</material>
+    </gazebo>
+    <gazebo reference="${prefix}link_proximal_actuating_bar">
+      <material>Gazebo/Black</material>
+    </gazebo>
+    <gazebo reference="${prefix}link_paraproximal_bar">
+      <material>Gazebo/Black</material>
+    </gazebo>
+    <gazebo reference="${prefix}link_median_actuating_hinge">
+      <material>Gazebo/Black</material>
+    </gazebo>
+    <gazebo reference="${prefix}link_median_bar">
+      <material>Gazebo/Black</material>
+    </gazebo>
+    <gazebo reference="${prefix}link_paramedian_hinge">
+      <material>Gazebo/Black</material>
+    </gazebo>
+    <gazebo reference="${prefix}link_median_bar_underactuated">
+      <material>Gazebo/Black</material>
+    </gazebo>
+    <gazebo reference="${prefix}link_paradistal_hinge">
+      <material>Gazebo/Black</material>
     </gazebo>
   </xacro:macro>
@@ -715,4 +755,8 @@
     </gazebo>
     <!-- end of joint list -->
+    <!-- Adding color for Gazebo visualization -->
+    <gazebo reference="${prefix}palm">
+      <material>Gazebo/Black</material>
+    </gazebo>
   </xacro:macro>
 </robot>

Commit message: Changed hand color in Rviz from green to black

File: robotiq_s_model_visualization/cfg/robotiq_hand_macro.urdf.xacro (robot description, xacro)
@@ -16,6 +16,6 @@
           <mesh filename="package://robotiq_s_model_visualization/meshes/s-model_articulated/visual/link_0.STL" />
         </geometry>
-        <material name="green">
-          <color rgba="0 1 0 1"/>
+        <material name="black"> <!-- green -->
+          <color rgba="0.0.5 0.05 0.05 1"/>
         </material>
       </visual>
@@ -46,5 +46,5 @@
           <mesh filename="package://robotiq_s_model_visualization/meshes/s-model_articulated/visual/link_1.STL" />
         </geometry>
-        <material name="green"/>
+        <material name="black"/> <!-- green -->
       </visual>
       <collision>
@@ -79,5 +79,5 @@
           <mesh filename="package://robotiq_s_model_visualization/meshes/s-model_articulated/visual/link_2.STL" />
         </geometry>
-        <material name="green"/>
+        <material name="black"/> <!-- green -->
       </visual>
       <collision>
@@ -110,5 +110,5 @@
           <mesh filename="package://robotiq_s_model_visualization/meshes/s-model_articulated/visual/link_3.STL" />
         </geometry>
-        <material name="green"/>
+        <material name="black"/> <!-- green -->
       </visual>
       <collision>
@@ -690,5 +690,5 @@
             <mesh filename="package://robotiq_s_model_visualization/meshes/s-model_articulated/visual/palm.STL" />
           </geometry>
-          <material name="green">
+          <material name="black"> <!-- yellow -->
             <color rgba="0 1 0 1"/>
           </material>

Commit message: Temporarily commented out collision of the underactuated red links while finishing the srdf

File: robotiq_s_model_visualization/cfg/robotiq_hand_macro.urdf.xacro (robot description, xacro)
@@ -142,10 +142,10 @@
         </geometry>
       </visual>
-      <collision>
+ <!--     <collision>
         <origin rpy="0 0 0" xyz="0.01429 0 0"/>
          <geometry>
           <box size="0.02858 .0075 .002"/>
         </geometry>
-      </collision>
+      </collision>-->
       <inertial>
         <origin rpy="0 0 0" xyz="0.0012 -0.00162 -0.00161"/>
@@ -171,10 +171,10 @@
         </geometry>
       </visual>
-      <collision>
+   <!--   <collision>
         <origin rpy="0 0 0" xyz="0.01143 0 0"/>
          <geometry>
           <box size="0.02286 .0075 .002"/>
         </geometry>
-      </collision>
+      </collision>-->
       <inertial>
         <origin rpy="0 0 0" xyz="0.0064 0 0"/>
@@ -201,10 +201,10 @@
         </geometry>
       </visual>
-      <collision>
+ <!--     <collision>
         <origin rpy="0 0 0" xyz="0.026789 0 0"/>
          <geometry>
           <box size="0.05398 .0075 .002"/>
         </geometry>
-      </collision>
+      </collision>-->
       <inertial>
         <origin rpy="0 0 0" xyz="0.02699 -0.00122 0"/>
@@ -230,10 +230,10 @@
         </geometry>
       </visual>
-      <collision>
+<!--      <collision>
         <origin rpy="0 0 0" xyz="0.02885 0 0"/>
          <geometry>
           <box size="0.05770 .0075 .002"/>
         </geometry>
-      </collision>
+      </collision>-->
       <inertial>
         <origin rpy="0 0 0" xyz="0.02858 -0.00129 0"/>
@@ -259,10 +259,10 @@
         </geometry>
       </visual>
-      <collision>
+<!--      <collision>
         <origin rpy="0 0 0" xyz="0 0 0"/>
          <geometry>
           <box size=".02 .02 .002"/>
         </geometry>
-      </collision>
+      </collision>-->
       <inertial>
         <origin rpy="0 0 0" xyz="0.0092 0.00514 0"/>
@@ -288,10 +288,10 @@
         </geometry>
       </visual>
-      <collision>
+<!--      <collision>
         <origin rpy="0 0 0" xyz="0.01905 0 0"/>
          <geometry>
           <box size="0.0381 .0075 .002"/>
         </geometry>
-      </collision>
+      </collision>-->
       <inertial>
         <origin rpy="0 0 0" xyz="0.01905 -0.00107 0"/>
@@ -317,10 +317,10 @@
         </geometry>
       </visual>
-      <collision>
+<!--      <collision>
         <origin rpy="0 0 0" xyz="0 0 0"/>
          <geometry>
           <box size=".02 .02 .002"/>
         </geometry>
-      </collision>
+      </collision>-->
       <inertial>
         <origin rpy="0 0 0" xyz="-0.01025 0.00046 0"/>
@@ -346,10 +346,10 @@
         </geometry>
       </visual>
-      <collision>
+  <!--    <collision>
         <origin rpy="0 0 0" xyz="0.01905 0 0"/>
          <geometry>
           <box size="0.0381 .0075 .002"/>
         </geometry>
-      </collision>
+      </collision>-->
       <inertial>
         <origin rpy="0 0 0" xyz="0.01905 -0.00107 0"/>
@@ -375,10 +375,10 @@
         </geometry>
       </visual>
-      <collision>
+  <!--    <collision>
         <origin rpy="0 0 0" xyz="0 0 0"/>
          <geometry>
           <box size=".02 0.02 .002"/>
         </geometry>
-      </collision>
+      </collision>-->
       <inertial>
         <origin rpy="0 0 0" xyz="0.00548 0 0"/>
